File: a.brd (EAGLE design)
At the start: 50 x 42.2 mm, 29 parts, among them CON1 PINHEAD_1X04-2.54, CON2 PINHEAD_1X08-2.54, CON3 PINHEAD_1X05-2, CON4 PINHEAD_2X03-PTH-2.54, SW1 TACT_SWITCH-1-1825910-4, SW2 TACT_SWITCH-1-1825910-4

Commit message: silk fixes
Parts:
- renumbered CON3 to X3, CON4 to X4
Other:
- board text added: "26.02.2026"
- board text added: "EBUCCCI reDesign"
- board text added: "JTAG"
- board text added: "PROG"
- board text added: "pds019_485_010a"

Commit message: readme
Changed lines of the file:
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@@
 <setting verticaltext="up"/>
 </settings>
-<grid distance="0.25" unitdist="mm" unit="mm" style="lines" multiple="1" display="yes" altdistance="0.05" altunitdist="mm" altunit="mm"/>
+<grid distance="0.1" unitdist="mm" unit="mm" style="lines" multiple="1" display="yes" altdistance="0.05" altunitdist="mm" altunit="mm"/>
 <layers>
 <layer number="1" name="Top" color="4" fill="1" visible="yes" active="yes"/>
@@
 </layers>
 <board>
-<fusionsync huburn="a.YnVzaW5lc3M6Z21haWw1NzY2MDI" projecturn="a.YnVzaW5lc3M6Z21haWw1NzY2MDIjMjAyNTA2MzA5NDU5NzA2ODE" f3durn="urn:adsk.wipprod:dm.lineage:iXZQqLShTUeB7U-ikoiT2A" pcbguid="" lastpulledtime="" lastsyncedchangeguid="" latestrevisionid="c897eee5-9ea5-4e3c-a58b-7956c222f2be" lastsyncedrevisionid="c897eee5-9ea5-4e3c-a58b-7956c222f2be" lastboardhashguid="e7db7193-5034-6e82-ccf8-01d87fa10b49" lastpushedtime="2026-02-25T18:09:42Z" linktopcb3d="false"/>
+<fusionsync huburn="a.YnVzaW5lc3M6Z21haWw1NzY2MDI" projecturn="a.YnVzaW5lc3M6Z21haWw1NzY2MDIjMjAyNTA2MzA5NDU5NzA2ODE" f3durn="urn:adsk.wipprod:dm.lineage:iXZQqLShTUeB7U-ikoiT2A" pcbguid="" lastpulledtime="" lastsyncedchangeguid="" latestrevisionid="27153e8c-3ebf-4b2a-a7d0-13bb084ce08d" lastsyncedrevisionid="27153e8c-3ebf-4b2a-a7d0-13bb084ce08d" lastboardhashguid="b2e55312-8973-685c-e83c-c5cf1c540762" lastpushedtime="2026-02-26T17:54:01Z" linktopcb3d="true"/>
 <plain>
 <wire x1="6.605440625" y1="13.780053125" x2="6.2037125" y2="14.18178125" width="0.082475" layer="48"/>
@@
 <text x="32.25" y="15.5" size="1.5" layer="21" font="vector" ratio="12">EBUCCCI
 reDesign</text>
+<wire x1="16.9" y1="4.4" x2="16.9" y2="1.7" width="0.5" layer="21"/>
+<wire x1="16.9" y1="1.7" x2="17" y2="1.6" width="0.5" layer="21"/>
+<wire x1="17" y1="1.6" x2="19.5" y2="1.6" width="0.5" layer="21"/>
+<wire x1="28.5" y1="4.2" x2="28.5" y2="2" width="0.5" layer="21"/>
+<wire x1="28.5" y1="2" x2="28.6" y2="1.9" width="0.5" layer="21"/>
+<wire x1="28.6" y1="1.9" x2="30.6" y2="1.9" width="0.5" layer="21"/>
 </plain>
 <attributes>
@@
 </element>
 <element name="X3" library="pinhead" library_urn="urn:adsk.eagle:library:2540341" package="1X05-PTH-2" package3d_urn="urn:adsk.eagle:package:4854339/2" value="PINHEAD_1X05-2" x="33.91" y="3.31" smashed="yes">
-<attribute name="NAME" x="30.25" y="1.5" size="1" layer="25" font="vector" ratio="15" align="center"/>
+<attribute name="NAME" x="31.75" y="1.5" size="1" layer="25" font="vector" ratio="15" align="center"/>
 </element>
 <element name="X4" library="pinhead" library_urn="urn:adsk.eagle:library:2540341" package="2X03-PTH-2.54" package3d_urn="urn:adsk.eagle:package:8729607/3" value="PINHEAD_2X03-PTH-2.54" x="21.2" y="4.55" smashed="yes" rot="R90">
