File: a.brd (EAGLE design)
At the start: 50 x 42.2 mm, 29 parts, among them CON1 PINHEAD_1X04-2.54, CON2 PINHEAD_1X08-2.54, SW1 TACT_SWITCH-1-1825910-4, SW2 TACT_SWITCH-1-1825910-4, X3 PINHEAD_1X05-2, X4 PINHEAD_2X03-PTH-2.54

Commit message: A pcb updates
Parts:
- removed HL1: LED_RGB-3528, rc:LED3528
- removed HL2, HL3: LED-0805, rc:LED0805
- added LED1, LED2, LED3: LED_RGB-3528, rc:LED3528
- added R15: 1K, rc:R0805
- added R17: 100R, rc:R0805
- R10, R9: value 470R -> 1K
- R6: value 3K3 -> 1K
- R7: value 8K2 -> 1K
- R8: value 12K -> 1K
- X3: value PINHEAD_1X05-2 -> PINHEAD_1X06-2-MALE; device pinhead:1X05-PTH-2 -> pinhead:1X06-PTH-2
- moved R6 10.1 mm to (3.50, 29.0)
- moved R10 8.46 mm to (3.50, 37.0), turned to 0 degrees
- moved R8 4.74 mm to (3.50, 33.0)
- moved R5 4.37 mm to (45.0, 5.50)
- moved R7 3.28 mm to (3.50, 35.0)
- moved R4 3.01 mm to (43.0, 3.50)
- moved R9 1.93 mm to (3.50, 31.0)
- moved X3 0.84 mm to (34.8, 3.25)
Connections:
- removed net !LED_B: MODULE1.24, R8.1
- removed net !LED_G: MODULE1.26, R7.1
- removed net !LED_IN: MODULE1.30, R9.1
- removed net !LED_OUT: MODULE1.31, R10.1
- removed net !LED_R: MODULE1.29, R6.1
- new net G1LED: MODULE1.31, R7.1
- new net G2LED: MODULE1.29, R9.1
- new net G3LED: MODULE1.24, R15.1
- new net N$11: LED3.4, R15.2
- new net N$17: R17.2, X3.1
- new net R1LED: MODULE1.33, R10.1
- new net R2LED: MODULE1.30, R8.1
- new net R3LED: MODULE1.26, R6.1
- net ESP_EN: now also R17.1
- net ESP_RXD0: now also R5.1; no longer R4.1
- net ESP_TXD0: now also R4.1; no longer R5.1
- net GND: now also X3.4; no longer X3.3
- net N$1: now also LED2.1; no longer HL1.4
- net N$10: now also LED3.1, R6.2; no longer HL1.3, R7.2
- net N$3: now also R5.2, X3.6; no longer R3.2, X3.2
- net N$4: now also X3.5; no longer X3.4
- net N$5: now also R3.2, X3.3; no longer R5.2, X3.5
- net N$7: now also LED1.1, R10.2; no longer HL2.C, R9.2
- net N$8: now also LED1.4, R7.2; no longer HL3.C, R10.2
- net N$9: now also LED2.4, R9.2; no longer HL1.1, R6.2
- net VDD_3V3: now also LED1.2, LED2.2, LED3.2, X3.2; no longer HL1.2, HL2.A, HL3.A, X3.1
Routing:
- net !LED_B: track 64.8 -> 0.00 mm, vias 2 -> 0
- net !LED_G: track 58.6 -> 0.00 mm, vias 2 -> 0
- net !LED_R: track 57.9 -> 0.00 mm, vias 2 -> 0
- net G3LED: track 0.00 -> 57.8 mm, vias 0 -> 2
- net R3LED: track 0.00 -> 56.5 mm, vias 0 -> 2
- net G1LED: track 0.00 -> 54.4 mm, vias 0 -> 2
- net R2LED: track 0.00 -> 54.3 mm, vias 0 -> 2
- net G2LED: track 0.00 -> 54.1 mm, vias 0 -> 2
- net R1LED: track 0.00 -> 53.7 mm, vias 0 -> 2
- net !LED_IN: track 50.8 -> 0.00 mm, vias 2 -> 0
- net !LED_OUT: track 44.5 -> 0.00 mm, vias 2 -> 0
- net N$17: track 0.00 -> 15.3 mm
- net VDD_3V3: track 86.9 -> 95.7 mm
- net ESP_EN: track 37.0 -> 44.4 mm
- net N$5: track 2.36 -> 7.93 mm
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Other:
- board text added: "3.3"
- board text added: "BT"
- board text added: "EN"
- board text added: "G"
- board text added: "RX"
- board text added: "TX"
