File: b.sch (EAGLE design)
At the start: 64 parts, among them CN1 CON-2P-DG500-5.08, CN2 CON-3P-DG500-5.08, CN3 CON-2P-DG500-5.08, CN4 CON-3P-DG500-5.08, CN5 CON-2P-DG500-5.08, Q1 BCR133, U2 TPS563200, U3 ISO3082, U4 B1212S-1WR3, U5 L78L05ACD13TR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

Commit message: readme
Parts:
- F1: device tmp:MST1.6A250V-MST -> rc:FUSE-MST
Changed lines of the file:
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@@
 <part name="FRAME1" library="frames" library_urn="urn:adsk.eagle:library:229" deviceset="A4L-LOC" device=""/>
 <part name="D2" library="TVS_diodes" library_urn="urn:adsk.eagle:library:3333632" deviceset="SM712" device="" package3d_urn="urn:adsk.eagle:package:3333648/5"/>
-<part name="U5" library="linear regulators" library_urn="urn:adsk.eagle:library:2541155" deviceset="L78L05ACD13TR" device="" package3d_urn="urn:adsk.eagle:package:20898192/5"/>
+<part name="U5" library="linear regulators" library_urn="urn:adsk.eagle:library:2541155" deviceset="L78L05ACD13TR" device="" package3d_urn="urn:adsk.eagle:package:20898192/5" override_package3d_urn="urn:adsk.eagle:package:20898192/7" override_package_urn="urn:adsk.eagle:footprint:4771000/5"/>
 <part name="C10" library="rc" library_urn="urn:adsk.eagle:library:2539423" deviceset="C" device="-0805" package3d_urn="urn:adsk.eagle:package:2539460/3" value="10u"/>
 <part name="C11" library="rc" library_urn="urn:adsk.eagle:library:2539423" deviceset="C" device="-0805" package3d_urn="urn:adsk.eagle:package:2539460/3" value="1u"/>
@@
 <part name="L5" library="rc" library_urn="urn:adsk.eagle:library:2539423" deviceset="L" device="-0805" package3d_urn="urn:adsk.eagle:package:32710307/2"/>
 <part name="GND14" library="supply_symbols" library_urn="urn:adsk.eagle:library:5017758" deviceset="GNDD" device="" value="GNDD"/>
-<part name="MODULE2" library="ac-dc" library_urn="urn:adsk.eagle:library:51565678" deviceset="IRM-05-12" device="" package3d_urn="urn:adsk.eagle:package:52043181/1"/>
+<part name="MODULE2" library="ac-dc" library_urn="urn:adsk.eagle:library:51565678" deviceset="IRM-05-12" device="" package3d_urn="urn:adsk.eagle:package:52043181/2"/>
 <part name="R1" library="rc" library_urn="urn:adsk.eagle:library:2539423" deviceset="R" device="-1206" package3d_urn="urn:adsk.eagle:package:2539464/2" technology="-1%" value="10R"/>
-<part name="F1" library="tmp" deviceset="MST1.6A250V" device="-MST" value="1.6A">
+<part name="F1" library="rc" library_urn="urn:adsk.eagle:library:2539423" deviceset="FUSE" device="-MST" value="1.6A">
 <attribute name="PACKAGE" value="PBF-4"/>
 </part>
@@
 packages will not be understood (or retained) with this version.
 </note>
+<note version="9.4" severity="warning">
+Since Version 9.4, EAGLE supports the overriding of 3D packages
+in schematics and board files. Those overridden 3d packages
+will not be understood (or retained) with this version.
+</note>
 </compatibility>
