File: a.sch (EAGLE design)
At the start: 28 parts, among them CON1 PINHEAD_1X04-2.54, CON2 PINHEAD_1X08-2.54, CON3 PINHEAD_1X05-2, CON4 PINHEAD_2X03-PTH-2.54, SW1 TACT_SWITCH-1-1825910-4, SW2 TACT_SWITCH-1-1825910-4

Commit message: silk fixes
Parts:
- renumbered CON3 to X3, CON4 to X4
Changed lines of the file:
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@@
 <part name="+P4" library="supply_symbols" library_urn="urn:adsk.eagle:library:5017758" deviceset="3.3V" device=""/>
 <part name="GND6" library="supply_symbols" library_urn="urn:adsk.eagle:library:5017758" deviceset="GND" device="" value="GND"/>
-<part name="CON3" library="pinhead" library_urn="urn:adsk.eagle:library:2540341" deviceset="PINHEAD_1X05" device="-2" package3d_urn="urn:adsk.eagle:package:4854339/2"/>
+<part name="X3" library="pinhead" library_urn="urn:adsk.eagle:library:2540341" deviceset="PINHEAD_1X05" device="-2" package3d_urn="urn:adsk.eagle:package:4854339/2"/>
 <part name="+P5" library="supply_symbols" library_urn="urn:adsk.eagle:library:5017758" deviceset="3.3V" device=""/>
 <part name="GND7" library="supply_symbols" library_urn="urn:adsk.eagle:library:5017758" deviceset="GND" device="" value="GND"/>
@@
 <part name="R4" library="rc" library_urn="urn:adsk.eagle:library:2539423" deviceset="R" device="-0805" package3d_urn="urn:adsk.eagle:package:2539455/2" technology="-1%" value="43R"/>
 <part name="R5" library="rc" library_urn="urn:adsk.eagle:library:2539423" deviceset="R" device="-0805" package3d_urn="urn:adsk.eagle:package:2539455/2" technology="-1%" value="43R"/>
-<part name="CON4" library="pinhead" library_urn="urn:adsk.eagle:library:2540341" deviceset="PINHEAD_2X03" device="-PTH-2.54" package3d_urn="urn:adsk.eagle:package:8729607/3"/>
+<part name="X4" library="pinhead" library_urn="urn:adsk.eagle:library:2540341" deviceset="PINHEAD_2X03" device="-PTH-2.54" package3d_urn="urn:adsk.eagle:package:8729607/3"/>
 <part name="+P6" library="supply_symbols" library_urn="urn:adsk.eagle:library:5017758" deviceset="3.3V" device=""/>
 <part name="GND8" library="supply_symbols" library_urn="urn:adsk.eagle:library:5017758" deviceset="GND" device="" value="GND"/>
@@
 <attribute name="VALUE" x="68.58" y="26.67" size="1.27" layer="96" font="vector" ratio="15" align="center"/>
 </instance>
-<instance part="CON3" gate="G$1" x="83.82" y="45.72" smashed="yes" rot="MR180">
+<instance part="X3" gate="G$1" x="83.82" y="45.72" smashed="yes" rot="MR180">
 <attribute name="NAME" x="86.36" y="29.21" size="1.778" layer="95" font="vector" ratio="15" rot="MR180" align="center"/>
 </instance>
@@
 <attribute name="ALLOCATED" x="99.06" y="31.496" size="0.762" layer="97" font="vector" rot="R180" align="center"/>
 </instance>
-<instance part="CON4" gate="G$1" x="114.3" y="66.04" smashed="yes">
+<instance part="X4" gate="G$1" x="114.3" y="66.04" smashed="yes">
 <attribute name="NAME" x="120.904" y="77.47" size="1.778" layer="95" font="vector" ratio="15" align="center"/>
 </instance>
@@
 <segment>
 <pinref part="GND7" gate="1" pin="GND"/>
-<pinref part="CON3" gate="G$1" pin="3"/>
+<pinref part="X3" gate="G$1" pin="3"/>
 <wire x1="93.98" y1="38.1" x2="91.44" y2="38.1" width="0.1524" layer="91"/>
 </segment>
@@
 <pinref part="GND8" gate="1" pin="GND"/>
 <wire x1="132.08" y1="66.04" x2="132.08" y2="68.58" width="0.1524" layer="91"/>
-<pinref part="CON4" gate="G$1" pin="6"/>
+<pinref part="X4" gate="G$1" pin="6"/>
 <wire x1="132.08" y1="68.58" x2="129.54" y2="68.58" width="0.1524" layer="91"/>
 </segment>
@@
 </segment>
 <segment>
-<pinref part="CON3" gate="G$1" pin="1"/>
+<pinref part="X3" gate="G$1" pin="1"/>
 <wire x1="91.44" y1="43.18" x2="93.98" y2="43.18" width="0.1524" layer="91"/>
 <pinref part="+P5" gate="G$1" pin="VDD_3V3"/>
@@
 </segment>
 <segment>
-<pinref part="CON4" gate="G$1" pin="1"/>
+<pinref part="X4" gate="G$1" pin="1"/>
 <wire x1="111.76" y1="73.66" x2="109.22" y2="73.66" width="0.1524" layer="91"/>
 <pinref part="+P6" gate="G$1" pin="VDD_3V3"/>
@@
 <net name="N$3" class="0">
 <segment>
-<pinref part="CON3" gate="G$1" pin="2"/>
+<pinref part="X3" gate="G$1" pin="2"/>
 <wire x1="91.44" y1="40.64" x2="99.06" y2="40.64" width="0.1524" layer="91"/>
 <pinref part="R3" gate="G$1" pin="2"/>
@@
 <net name="N$4" class="0">
 <segment>
-<pinref part="CON3" gate="G$1" pin="4"/>
+<pinref part="X3" gate="G$1" pin="4"/>
 <wire x1="91.44" y1="35.56" x2="99.06" y2="35.56" width="0.1524" layer="91"/>
 <pinref part="R4" gate="G$1" pin="2"/>
@@
 <net name="N$5" class="0">
 <segment>
-<pinref part="CON3" gate="G$1" pin="5"/>
+<pinref part="X3" gate="G$1" pin="5"/>
 <wire x1="91.44" y1="33.02" x2="93.98" y2="33.02" width="0.1524" layer="91"/>
 <pinref part="R5" gate="G$1" pin="2"/>
@@
 <net name="N$2" class="0">
 <segment>
-<pinref part="CON4" gate="G$1" pin="2"/>
+<pinref part="X4" gate="G$1" pin="2"/>
 <wire x1="129.54" y1="73.66" x2="139.7" y2="73.66" width="0.1524" layer="91"/>
 <pinref part="R13" gate="G$1" pin="2"/>
@@
 <segment>
 <pinref part="R12" gate="G$1" pin="2"/>
-<pinref part="CON4" gate="G$1" pin="4"/>
+<pinref part="X4" gate="G$1" pin="4"/>
 <wire x1="132.08" y1="71.12" x2="129.54" y2="71.12" width="0.1524" layer="91"/>
 </segment>
@@
 <segment>
 <pinref part="R14" gate="G$1" pin="1"/>
-<pinref part="CON4" gate="G$1" pin="3"/>
+<pinref part="X4" gate="G$1" pin="3"/>
 <wire x1="109.22" y1="71.12" x2="111.76" y2="71.12" width="0.1524" layer="91"/>
 </segment>
@@
 <net name="N$15" class="0">
 <segment>
-<pinref part="CON4" gate="G$1" pin="5"/>
+<pinref part="X4" gate="G$1" pin="5"/>
 <pinref part="R11" gate="G$1" pin="1"/>
 <wire x1="111.76" y1="68.58" x2="101.6" y2="68.58" width="0.1524" layer="91"/>

Commit message: A pcb updates
Parts:
- removed HL1: LED_RGB-3528, rc:LED_RGB-3528
- removed HL2, HL3: LED-0805, rc:LED-0805
- added LED1, LED2, LED3: LED_RGB-3528, rc:LED_RGB-3528
- added R15: 1K, rc:R-1%-0805
- added R17: 100R, rc:R-1%-0805
- R10, R9: value 470R -> 1K
- R6: value 3K3 -> 1K
- R7: value 8K2 -> 1K
- R8: value 12K -> 1K
- X3: value PINHEAD_1X05-2 -> PINHEAD_1X06-2-MALE; device pinhead:PINHEAD_1X05-2 -> pinhead:PINHEAD_1X06-2-MALE
Connections:
- removed net !LED_B: MODULE1.IO2, R8.1
- removed net !LED_G: MODULE1.IO4, R7.1
- removed net !LED_IN: MODULE1.IO18, R9.1
- removed net !LED_OUT: MODULE1.IO19, R10.1
- removed net !LED_R: MODULE1.IO5, R6.1
- new net G1LED: MODULE1.IO19, R7.1
- new net G2LED: MODULE1.IO5, R9.1
- new net G3LED: MODULE1.IO2, R15.1
- new net N$11: LED3.G, R15.2
- new net N$17: R17.2, X3.1
- new net R1LED: MODULE1.IO21, R10.1
- new net R2LED: MODULE1.IO18, R8.1
- new net R3LED: MODULE1.IO4, R6.1
- net ESP_EN: now also R17.1
- net ESP_RXD0: now also R5.1; no longer R4.1
- net ESP_TXD0: now also R4.1; no longer R5.1
- net GND: now also X3.4; no longer X3.3
- net N$1: now also LED2.R; no longer HL1.G
- net N$10: now also LED3.R, R6.2; no longer HL1.B, R7.2
- net N$3: now also R5.2, X3.6; no longer R3.2, X3.2
- net N$4: now also X3.5; no longer X3.4
- net N$5: now also R3.2, X3.3; no longer R5.2, X3.5
- net N$7: now also LED1.R, R10.2; no longer HL2.C, R9.2
- net N$8: now also LED1.G, R7.2; no longer HL3.C, R10.2
- net N$9: now also LED2.G, R9.2; no longer HL1.R, R6.2
- net VDD_3V3: now also LED1.A, LED2.A, LED3.A, X3.2; no longer HL1.A, HL2.A, HL3.A, X3.1
Other:
- moved on the sheet: R10, R3, R4, R5, R6, R7, R8, R9
